Commit message: add web dashboard

File: install/autonomous_explorer/share/autonomous_explorer/urdf/explorer_bot.urdf.xacro (robot description, xacro)
@@ -1 +1,261 @@
-/home/sanket/robot_mapping_ws/build/autonomous_explorer/urdf/explorer_bot.urdf.xacro
+<?xml version="1.0"?>
+<robot xmlns:xacro="http://www.ros.org/wiki/xacro" name="mecanum_robot">
+  <!-- Define properties based on your CAD model -->
+  <xacro:property name="base_length" value="0.7"/>  <!-- 700mm -->
+  <xacro:property name="base_width" value="0.45"/>   <!-- 450mm -->
+  <xacro:property name="base_height" value="0.18"/>  <!-- 180mm -->
+  <!-- Mecanum wheel properties -->
+  <xacro:property name="wheel_radius" value="0.1"/>  <!-- 100mm radius = 200mm diameter -->
+  <xacro:property name="wheel_width" value="0.07"/>  <!-- 70mm width -->
+  <xacro:property name="wheelbase" value="0.5"/>     <!-- 500mm front to back -->
+  <xacro:property name="track_width" value="0.425"/> <!-- 425mm left to right -->
+  <!-- Lifting arm properties -->
+  <xacro:property name="arm_length" value="0.6"/>    <!-- 600mm -->
+  <xacro:property name="arm_width" value="0.325"/>   <!-- 325mm -->
+  <xacro:property name="arm_height" value="0.1"/>    <!-- 100mm -->
+  <!-- Base Footprint -->
+  <link name="base_footprint"/>
+  <!-- Base Link (Main Chassis) -->
+  <link name="base_link">
+    <visual>
+      <geometry>
+        <box size="${base_length} ${base_width} ${base_height}"/>
+      </geometry>
+      <material name="dark_grey">
+        <color rgba="0.3 0.3 0.3 1"/>
+      </material>
+    </visual>
+    <collision>
+      <geometry>
+        <box size="${base_length} ${base_width} ${base_height}"/>
+      </geometry>
+    </collision>
+    <inertial>
+      <mass value="15.0"/>  <!-- Heavier base for your robot -->
+      <inertia ixx="0.5" ixy="0.0" ixz="0.0" iyy="0.8" iyz="0.0" izz="1.0"/>
+    </inertial>
+  </link>
+  <joint name="base_joint" type="fixed">
+    <parent link="base_footprint"/>
+    <child link="base_link"/>
+    <origin xyz="0 0 ${wheel_radius}" rpy="0 0 0"/>
+  </joint>
+  <!-- Mecanum Wheels Macro -->
+  <xacro:macro name="mecanum_wheel" params="prefix reflect_x reflect_y">
+    <link name="${prefix}_wheel">
+      <visual>
+        <geometry>
+          <cylinder radius="${wheel_radius}" length="${wheel_width}"/>
+        </geometry>
+        <material name="black">
+          <color rgba="0.1 0.1 0.1 1"/>
+        </material>
+      </visual>
+      <collision>
+        <geometry>
+          <cylinder radius="${wheel_radius}" length="${wheel_width}"/>
+        </geometry>
+      </collision>
+      <inertial>
+        <mass value="1.5"/>
+        <inertia ixx="0.01" ixy="0.0" ixz="0.0" iyy="0.01" iyz="0.0" izz="0.015"/>
+      </inertial>
+    </link>
+    <joint name="${prefix}_wheel_joint" type="continuous">
+      <parent link="base_link"/>
+      <child link="${prefix}_wheel"/>
+      <origin xyz="${reflect_x*wheelbase/2} ${reflect_y*track_width/2} 0" rpy="-1.5707 0 0"/>
+      <axis xyz="0 0 1"/>
+    </joint>
+  </xacro:macro>
+  <!-- Create 4 mecanum wheels -->
+  <xacro:mecanum_wheel prefix="front_left" reflect_x="1" reflect_y="1"/>
+  <xacro:mecanum_wheel prefix="front_right" reflect_x="1" reflect_y="-1"/>
+  <xacro:mecanum_wheel prefix="rear_left" reflect_x="-1" reflect_y="1"/>
+  <xacro:mecanum_wheel prefix="rear_right" reflect_x="-1" reflect_y="-1"/>
+  <!-- Lifting Arm Base -->
+  <link name="arm_base">
+    <visual>
+      <geometry>
+        <box size="${arm_length} ${arm_width} ${arm_height}"/>
+      </geometry>
+      <material name="orange">
+        <color rgba="1.0 0.5 0.0 1"/>
+      </material>
+    </visual>
+    <collision>
+      <geometry>
+        <box size="${arm_length} ${arm_width} ${arm_height}"/>
+      </geometry>
+    </collision>
+    <inertial>
+      <mass value="2.0"/>
+      <inertia ixx="0.02" ixy="0.0" ixz="0.0" iyy="0.06" iyz="0.0" izz="0.06"/>
+    </inertial>
+  </link>
+  <joint name="arm_base_joint" type="fixed">
+    <parent link="base_link"/>
+    <child link="arm_base"/>
+    <origin xyz="0.1 0 ${base_height/2 + arm_height/2 + 0.05}" rpy="0 0 0"/>
+  </joint>
+  <!-- LiDAR Sensor (mounted on top) -->
+  <link name="laser_link">
+    <visual>
+      <geometry>
+        <cylinder radius="0.05" length="0.07"/>
+      </geometry>
+      <material name="red">
+        <color rgba="1 0 0 1"/>
+      </material>
+    </visual>
+    <collision>
+      <geometry>
+        <cylinder radius="0.05" length="0.07"/>
+      </geometry>
+    </collision>
+    <inertial>
+      <mass value="0.2"/>
+      <inertia ixx="0.0001" ixy="0.0" ixz="0.0" iyy="0.0001" iyz="0.0" izz="0.0001"/>
+    </inertial>
+  </link>
+  <joint name="laser_joint" type="fixed">
+    <parent link="base_link"/>
+    <child link="laser_link"/>
+    <origin xyz="0.25 0 ${base_height/2 + 0.1}" rpy="0 0 0"/>
+  </joint>
+  <!-- Camera (USB Camera) -->
+  <link name="camera_link">
+    <visual>
+      <geometry>
+        <box size="0.03 0.1 0.03"/>
+      </geometry>
+      <material name="blue">
+        <color rgba="0 0 0.8 1"/>
+      </material>
+    </visual>
+    <collision>
+      <geometry>
+        <box size="0.03 0.1 0.03"/>
+      </geometry>
+    </collision>
+    <inertial>
+      <mass value="0.1"/>
+      <inertia ixx="0.0001" ixy="0.0" ixz="0.0" iyy="0.0001" iyz="0.0" izz="0.0001"/>
+    </inertial>
+  </link>
+  <joint name="camera_joint" type="fixed">
+    <parent link="arm_base"/>
+    <child link="camera_link"/>
+    <origin xyz="${arm_length/2 - 0.05} 0 ${arm_height/2 + 0.02}" rpy="0 0 0"/>
+  </joint>
+  <!-- Gazebo Plugins -->
+  <!-- Mecanum Drive Plugin -->
+  <gazebo>
+    <plugin name="mecanum_drive" filename="libgazebo_ros_planar_move.so">
+      <update_rate>50</update_rate>
+      <command_topic>cmd_vel</command_topic>
+      <odometry_topic>odom</odometry_topic>
+      <odometry_frame>odom</odometry_frame>
+      <odometry_rate>50.0</odometry_rate>
+      <robot_base_frame>base_footprint</robot_base_frame>
+      <publish_odom>true</publish_odom>
+      <publish_odom_tf>true</publish_odom_tf>
+    </plugin>
+  </gazebo>
+  <!-- LiDAR Plugin -->
+  <gazebo reference="laser_link">
+    <sensor name="laser_sensor" type="ray">
+      <pose>0 0 0 0 0 0</pose>
+      <visualize>true</visualize>
+      <update_rate>10</update_rate>
+      <ray>
+        <scan>
+          <horizontal>
+            <samples>360</samples>
+            <resolution>1</resolution>
+            <min_angle>-3.14159</min_angle>
+            <max_angle>3.14159</max_angle>
+          </horizontal>
+        </scan>
+        <range>
+          <min>0.2</min>
+          <max>10.0</max>
+          <resolution>0.01</resolution>
+        </range>
+        <noise>
+          <type>gaussian</type>
+          <mean>0.0</mean>
+          <stddev>0.01</stddev>
+        </noise>
+      </ray>
+      <plugin name="laser_controller" filename="libgazebo_ros_ray_sensor.so">
+        <ros>
+          <namespace>/</namespace>
+          <remapping>~/out:=scan</remapping>
+        </ros>
+        <output_type>sensor_msgs/LaserScan</output_type>
+        <frame_name>laser_link</frame_name>
+      </plugin>
+    </sensor>
+  </gazebo>
+  <!-- Camera Plugin -->
+  <gazebo reference="camera_link">
+    <sensor name="camera" type="camera">
+      <update_rate>30</update_rate>
+      <camera>
+        <horizontal_fov>1.047</horizontal_fov>
+        <image>
+          <width>640</width>
+          <height>480</height>
+          <format>R8G8B8</format>
+        </image>
+        <clip>
+          <near>0.05</near>
+          <far>10</far>
+        </clip>
+      </camera>
+      <plugin name="camera_controller" filename="libgazebo_ros_camera.so">
+        <ros>
+          <namespace>/</namespace>
+          <remapping>image_raw:=camera/image_raw</remapping>
+          <remapping>camera_info:=camera/camera_info</remapping>
+        </ros>
+        <camera_name>camera</camera_name>
+        <frame_name>camera_link</frame_name>
+      </plugin>
+    </sensor>
+  </gazebo>
+  <!-- Gazebo colors -->
+  <gazebo reference="base_link">
+    <material>Gazebo/DarkGrey</material>
+  </gazebo>
+  <gazebo reference="front_left_wheel">
+    <material>Gazebo/Black</material>
+    <mu1>0.8</mu1>
+    <mu2>0.8</mu2>
+  </gazebo>
+  <gazebo reference="front_right_wheel">
+    <material>Gazebo/Black</material>
+    <mu1>0.8</mu1>
+    <mu2>0.8</mu2>
+  </gazebo>
+  <gazebo reference="rear_left_wheel">
+    <material>Gazebo/Black</material>
+    <mu1>0.8</mu1>
+    <mu2>0.8</mu2>
+  </gazebo>
+  <gazebo reference="rear_right_wheel">
+    <material>Gazebo/Black</material>
+    <mu1>0.8</mu1>
+    <mu2>0.8</mu2>
+  </gazebo>
+  <gazebo reference="arm_base">
+    <material>Gazebo/Orange</material>
+  </gazebo>
+  <gazebo reference="laser_link">
+    <material>Gazebo/Red</material>
+  </gazebo>
+  <gazebo reference="camera_link">
+    <material>Gazebo/Blue</material>
+  </gazebo>
+</robot>
